File: myhalf.sch (EAGLE design)
At the start: 0 parts

Commit message: pogo-mating pads placed, outline drawn
Parts:
- added GND, INT, SCL, SDA, V33, VCC: SMD_1.5MM, OMAT_IC:SMD_1.5MM
Connections:
- new net GND: GND.1
- new net I2C_SCL: SCL.1
- new net I2C_SDA: SDA.1
- new net INT: INT.1
- new net V33: V33.1
- new net VCC: VCC.1
