File: myhalf.sch (EAGLE design)
At the start: 6 parts

Commit message: some more work progress...
Parts:
- added C1, C2: (no value), rcl:C-EUC0603
- added D1: PCA9517-MSOP8, OMAT_IC:PCA9517
- added D2: AT24C02C-SOT23-5, Microchip_By_element14_Batch_1:24LC01BT-I/OT
- added N1: MCP1700T-1802E/TT, Microchip_By_element14_Batch_1:MCP1700T-1802E/TT
- added R1, R2: (no value), rcl:R-EU_R0603
Connections:
- removed net I2C_SCL: SCL.1
- removed net I2C_SDA: SDA.1
- removed net V33: V33.1
- new net +1V8: C2.1, D1.VCCA, D2.VCC, N1.VOUT
- new net +3V3: C1.1, D1.VCCB, N1.VIN, R1.2, R2.2, V33.1
- new net SCL_1V8: D1.SCLA, D2.SCL, SCL.1
- new net SCL_3V3: D1.SCLB, R1.1
- new net SDA_1V8: D1.SDAA, D2.SDA, SDA.1
- new net SDA_3V3: D1.SDAB, R2.1
- net GND: now also C1.2, C2.2, D1.GND, D2.VSS, D2.WP, N1.GND

Commit message: good night
Parts:
- added SCL_3V3, SDA_3V3, V18, _GND, _INT, _V33: SMD_1.5MM, OMAT_IC:SMD_1.5MM
- added U$1: DAFUG, dafug:DAFUG
Connections:
- net +1V8: now also V18.1
- net +3V3: now also _V33.1
- net GND: now also _GND.1
- net INT: now also _INT.1
- net SCL_3V3: now also SCL_3V3.1
- net SDA_3V3: now also SDA_3V3.1
Changed lines of the file:
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@@
 <part name="R2" library="rcl" deviceset="R-EU_" device="R0603"/>
 <part name="+3V3" library="supply1" deviceset="+3V3" device=""/>
+<part name="SCL_3V3" library="OMAT_IC" deviceset="SMD_1.5MM" device=""/>
+<part name="SDA_3V3" library="OMAT_IC" deviceset="SMD_1.5MM" device=""/>
+<part name="V18" library="OMAT_IC" deviceset="SMD_1.5MM" device=""/>
+<part name="_GND" library="OMAT_IC" deviceset="SMD_1.5MM" device=""/>
+<part name="_V33" library="OMAT_IC" deviceset="SMD_1.5MM" device=""/>
+<part name="GND6" library="supply1" deviceset="GND" device=""/>
+<part name="+3V4" library="supply1" deviceset="+3V3" device=""/>
+<part name="+1V4" library="supply1" deviceset="+1V8" device=""/>
+<part name="_INT" library="OMAT_IC" deviceset="SMD_1.5MM" device=""/>
+<part name="U$1" library="dafug" deviceset="DAFUG" device=""/>
 </parts>
 <sheets>
@@
 <instance part="R2" gate="G$1" x="241.3" y="50.8" rot="R90"/>
 <instance part="+3V3" gate="G$1" x="88.9" y="48.26"/>
+<instance part="SCL_3V3" gate="G$1" x="261.62" y="43.18" rot="R180"/>
+<instance part="SDA_3V3" gate="G$1" x="261.62" y="30.48" rot="R180"/>
+<instance part="V18" gate="G$1" x="261.62" y="81.28" rot="R180"/>
+<instance part="_GND" gate="G$1" x="261.62" y="17.78" rot="R180"/>
+<instance part="_V33" gate="G$1" x="261.62" y="68.58" rot="R180"/>
+<instance part="GND6" gate="1" x="246.38" y="10.16"/>
+<instance part="+3V4" gate="G$1" x="243.84" y="73.66"/>
+<instance part="+1V4" gate="G$1" x="243.84" y="86.36"/>
+<instance part="_INT" gate="G$1" x="261.62" y="-2.54" rot="R180"/>
+<instance part="U$1" gate="G$1" x="177.8" y="2.54"/>
 </instances>
 <busses>
@@
 <wire x1="50.8" y1="78.74" x2="81.28" y2="78.74" width="0.1524" layer="91"/>
 <label x="68.58" y="78.74" size="1.778" layer="95"/>
+</segment>
+<segment>
+<pinref part="_INT" gate="G$1" pin="1"/>
+<wire x1="254" y1="-2.54" x2="223.52" y2="-2.54" width="0.1524" layer="91"/>
+<label x="226.06" y="-2.54" size="1.778" layer="95"/>
 </segment>
 </net>
@@
 <pinref part="GND5" gate="1" pin="GND"/>
 </segment>
+<segment>
+<pinref part="_GND" gate="G$1" pin="1"/>
+<pinref part="GND6" gate="1" pin="GND"/>
+<wire x1="254" y1="17.78" x2="246.38" y2="17.78" width="0.1524" layer="91"/>
+<wire x1="246.38" y1="17.78" x2="246.38" y2="12.7" width="0.1524" layer="91"/>
+</segment>
 </net>
 <net name="+1V8" class="0">
@@
 <wire x1="220.98" y1="152.4" x2="215.9" y2="152.4" width="0.1524" layer="91"/>
 <junction x="215.9" y="152.4"/>
+</segment>
+<segment>
+<pinref part="V18" gate="G$1" pin="1"/>
+<pinref part="+1V4" gate="G$1" pin="+1V8"/>
+<wire x1="254" y1="81.28" x2="243.84" y2="81.28" width="0.1524" layer="91"/>
+<wire x1="243.84" y1="81.28" x2="243.84" y2="86.36" width="0.1524" layer="91"/>
 </segment>
 </net>
@@
 <wire x1="88.9" y1="40.64" x2="88.9" y2="45.72" width="0.1524" layer="91"/>
 </segment>
+<segment>
+<pinref part="_V33" gate="G$1" pin="1"/>
+<pinref part="+3V4" gate="G$1" pin="+3V3"/>
+<wire x1="254" y1="68.58" x2="243.84" y2="68.58" width="0.1524" layer="91"/>
+<wire x1="243.84" y1="68.58" x2="243.84" y2="71.12" width="0.1524" layer="91"/>
+</segment>
 </net>
 <net name="SCL_3V3" class="0">
@@
 <pinref part="R1" gate="G$1" pin="1"/>
 <wire x1="231.14" y1="43.18" x2="231.14" y2="45.72" width="0.1524" layer="91"/>
-<wire x1="231.14" y1="43.18" x2="248.92" y2="43.18" width="0.1524" layer="91"/>
+<wire x1="231.14" y1="43.18" x2="254" y2="43.18" width="0.1524" layer="91"/>
 <junction x="231.14" y="43.18"/>
+<pinref part="SCL_3V3" gate="G$1" pin="1"/>
 </segment>
 </net>
@@
 <wire x1="241.3" y1="38.1" x2="248.92" y2="38.1" width="0.1524" layer="91"/>
 <junction x="241.3" y="38.1"/>
-</segment>
-</net>
+<pinref part="SDA_3V3" gate="G$1" pin="1"/>
+<wire x1="254" y1="30.48" x2="248.92" y2="30.48" width="0.1524" layer="91"/>
+<wire x1="248.92" y1="30.48" x2="248.92" y2="38.1" width="0.1524" layer="91"/>
+</segment>
+</net>

Commit message: v1.10
Parts:
- removed SCL_3V3, SDA_3V3, V18, _GND, _INT, _V33: SMD_1.5MM, OMAT_IC:SMD_1.5MM
- added H1: (no value), OMAT_IC:LEDCHIP-LED0603
- added R3: 330, rcl:R-EU_R0603
- added X1: PIIKKIRIMA-10, OMAT_IC:PIIKKIRIMA-10
- R1, R2: value (none) -> 2K15
Connections:
- new net N$2: H1.A, R3.1
- net +1V8: now also X1.5; no longer V18.1
- net +3V3: now also R3.2, X1.2; no longer _V33.1
- net GND: now also H1.C, X1.1, X1.10; no longer _GND.1
- net INT: now also X1.6; no longer _INT.1
- net SCL_1V8: now also X1.7
- net SCL_3V3: now also X1.3; no longer SCL_3V3.1
- net SDA_1V8: now also X1.8
- net SDA_3V3: now also X1.4; no longer SDA_3V3.1
- net VCC: now also X1.9
Other:
- note added: "CONNECTION TO JOLLA"
- note added: "MY OTHER HALF V1.10 BREAKOUT BOARD"
- moved on the sheet: C1, C2, D2, N1
