File: myhalf.brd (EAGLE design)
At the start: 48 x 48 mm, 0 parts

Commit message: pogo-mating pads placed, outline drawn
Parts:
- added GND, INT, SCL, SDA, V33, VCC: SMD_1.5MM, OMAT_IC:SMD_ROUND_1.5MM
Connections:
- new net GND: GND.1
- new net I2C_SCL: SCL.1
- new net I2C_SDA: SDA.1
- new net INT: INT.1
- new net V33: V33.1
- new net VCC: VCC.1
Routing:
- added copper zone on layer 1, net GND
- added copper zone on layer 16, net GND
- added copper zone on layer 16, net N$1
Other:
- outline, holes or cut-outs redrawn
Changed lines of the file:
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@@
 <setting verticaltext="up"/>
 </settings>
-<grid distance="1" unitdist="mm" unit="mm" style="lines" multiple="1" display="no" altdistance="0.025" altunitdist="inch" altunit="inch"/>
+<grid distance="0.5" unitdist="mm" unit="mm" style="lines" multiple="1" display="no" altdistance="0.025" altunitdist="inch" altunit="inch"/>
 <layers>
 <layer number="1" name="Top" color="4" fill="1" visible="yes" active="yes"/>
@@
 <layer number="43" name="vRestrict" color="2" fill="10" visible="yes" active="yes"/>
 <layer number="44" name="Drills" color="7" fill="1" visible="no" active="yes"/>
-<layer number="45" name="Holes" color="7" fill="1" visible="no" active="yes"/>
+<layer number="45" name="Holes" color="7" fill="1" visible="yes" active="yes"/>
 <layer number="46" name="Milling" color="3" fill="1" visible="no" active="yes"/>
 <layer number="47" name="Measures" color="7" fill="1" visible="no" active="yes"/>
 <layer number="48" name="Document" color="7" fill="1" visible="yes" active="yes"/>
 <layer number="49" name="Reference" color="7" fill="1" visible="yes" active="yes"/>
+<layer number="50" name="dxf" color="7" fill="1" visible="no" active="no"/>
 <layer number="51" name="tDocu" color="7" fill="1" visible="yes" active="yes"/>
 <layer number="52" name="bDocu" color="7" fill="1" visible="yes" active="yes"/>
+<layer number="53" name="tGND_GNDA" color="7" fill="9" visible="no" active="no"/>
+<layer number="54" name="bGND_GNDA" color="1" fill="9" visible="no" active="no"/>
+<layer number="56" name="wert" color="7" fill="1" visible="no" active="no"/>
 <layer number="91" name="Nets" color="2" fill="1" visible="no" active="no"/>
 <layer number="92" name="Busses" color="1" fill="1" visible="no" active="no"/>
@@
 <layer number="97" name="Info" color="7" fill="1" visible="no" active="no"/>
 <layer number="98" name="Guide" color="6" fill="1" visible="no" active="no"/>
+<layer number="100" name="Muster" color="7" fill="1" visible="no" active="no"/>
+<layer number="101" name="Hidden" color="15" fill="1" visible="yes" active="yes"/>
+<layer number="102" name="Changes" color="12" fill="1" visible="yes" active="yes"/>
+<layer number="103" name="tMap" color="7" fill="1" visible="yes" active="yes"/>
+<layer number="104" name="Name" color="16" fill="1" visible="yes" active="yes"/>
+<layer number="105" name="tPlate" color="7" fill="1" visible="yes" active="yes"/>
+<layer number="106" name="bPlate" color="7" fill="1" visible="yes" active="yes"/>
+<layer number="107" name="Crop" color="7" fill="1" visible="yes" active="yes"/>
+<layer number="108" name="fp8" color="7" fill="1" visible="yes" active="yes"/>
+<layer number="109" name="fp9" color="7" fill="1" visible="yes" active="yes"/>
+<layer number="110" name="fp0" color="7" fill="1" visible="yes" active="yes"/>
+<layer number="116" name="Patch_BOT" color="9" fill="4" visible="yes" active="yes"/>
+<layer number="121" name="_tsilk" color="7" fill="1" visible="yes" active="yes"/>
+<layer number="122" name="_bsilk" color="7" fill="1" visible="yes" active="yes"/>
+<layer number="123" name="tTestmark" color="7" fill="1" visible="yes" active="yes"/>
+<layer number="124" name="bTestmark" color="7" fill="1" visible="yes" active="yes"/>
+<layer number="131" name="tAdjust" color="7" fill="1" visible="yes" active="yes"/>
+<layer number="132" name="bAdjust" color="7" fill="1" visible="yes" active="yes"/>
+<layer number="144" name="Drill_legend" color="7" fill="1" visible="yes" active="yes"/>
+<layer number="151" name="HeatSink" color="7" fill="1" visible="yes" active="yes"/>
+<layer number="199" name="Contour" color="7" fill="1" visible="yes" active="yes"/>
+<layer number="200" name="200bmp" color="1" fill="10" visible="yes" active="yes"/>
+<layer number="201" name="201bmp" color="2" fill="10" visible="yes" active="yes"/>
+<layer number="202" name="202bmp" color="3" fill="10" visible="yes" active="yes"/>
+<layer number="203" name="203bmp" color="4" fill="10" visible="yes" active="yes"/>
+<layer number="204" name="204bmp" color="5" fill="10" visible="yes" active="yes"/>
+<layer number="205" name="205bmp" color="6" fill="10" visible="yes" active="yes"/>
+<layer number="206" name="206bmp" color="7" fill="10" visible="yes" active="yes"/>
+<layer number="207" name="207bmp" color="8" fill="10" visible="yes" active="yes"/>
+<layer number="208" name="208bmp" color="9" fill="10" visible="yes" active="yes"/>
+<layer number="209" name="209bmp" color="7" fill="1" visible="yes" active="yes"/>
+<layer number="210" name="210bmp" color="7" fill="1" visible="yes" active="yes"/>
+<layer number="211" name="211bmp" color="7" fill="1" visible="yes" active="yes"/>
+<layer number="212" name="212bmp" color="7" fill="1" visible="yes" active="yes"/>
+<layer number="213" name="213bmp" color="7" fill="1" visible="yes" active="yes"/>
+<layer number="214" name="214bmp" color="7" fill="1" visible="yes" active="yes"/>
+<layer number="215" name="215bmp" color="7" fill="1" visible="yes" active="yes"/>
+<layer number="216" name="216bmp" color="7" fill="1" visible="yes" active="yes"/>
+<layer number="217" name="217bmp" color="7" fill="1" visible="yes" active="yes"/>
+<layer number="218" name="218bmp" color="7" fill="1" visible="yes" active="yes"/>
+<layer number="219" name="219bmp" color="7" fill="1" visible="yes" active="yes"/>
+<layer number="220" name="220bmp" color="7" fill="1" visible="yes" active="yes"/>
+<layer number="221" name="221bmp" color="7" fill="1" visible="yes" active="yes"/>
+<layer number="222" name="222bmp" color="7" fill="1" visible="yes" active="yes"/>
+<layer number="223" name="223bmp" color="7" fill="1" visible="yes" active="yes"/>
+<layer number="224" name="224bmp" color="7" fill="1" visible="yes" active="yes"/>
+<layer number="250" name="Descript" color="3" fill="1" visible="no" active="no"/>
+<layer number="251" name="SMDround" color="12" fill="11" visible="no" active="no"/>
+<layer number="254" name="cooling" color="7" fill="1" visible="yes" active="yes"/>
 </layers>
 <board>
@@
 <wire x1="48" y1="48" x2="0" y2="48" width="0" layer="20"/>
 <wire x1="0" y1="48" x2="0" y2="0" width="0" layer="20"/>
+<wire x1="18" y1="30" x2="28" y2="30" width="0" layer="20"/>
+<wire x1="28" y1="30" x2="28" y2="40" width="0" layer="20"/>
+<wire x1="28" y1="40" x2="18" y2="40" width="0" layer="20"/>
+<wire x1="18" y1="40" x2="18" y2="30" width="0" layer="20"/>
+<hole x="33.5" y="35" drill="4"/>
 </plain>
 <attributes>
@@
 </autorouter>
 <elements>
+<element name="INT" library="OMAT_IC" package="SMD_ROUND_1.5MM" value="SMD_1.5MM" x="45.3" y="27.3" smashed="yes" rot="MR0">
+<attribute name="NAME" x="43.8" y="26.8" size="1" layer="26" rot="MR0"/>
+</element>
+<element name="SDA" library="OMAT_IC" package="SMD_ROUND_1.5MM" value="SMD_1.5MM" x="45.3" y="16.76" smashed="yes" rot="MR0">
+<attribute name="NAME" x="43.8" y="16.26" size="1" layer="26" rot="MR0"/>
+</element>
+<element name="SCL" library="OMAT_IC" package="SMD_ROUND_1.5MM" value="SMD_1.5MM" x="45.3" y="12.26" smashed="yes" rot="MR0">
+<attribute name="NAME" x="43.8" y="11.76" size="1" layer="26" rot="MR0"/>
+</element>
+<element name="V33" library="OMAT_IC" package="SMD_ROUND_1.5MM" value="SMD_1.5MM" x="45.3" y="24.76" smashed="yes" rot="MR0">
+<attribute name="NAME" x="43.8" y="24.26" size="1" layer="26" rot="MR0"/>
+</element>
+<element name="VCC" library="OMAT_IC" package="SMD_ROUND_1.5MM" value="SMD_1.5MM" x="4.6" y="6.5" smashed="yes" rot="MR0">
+<attribute name="NAME" x="4" y="7.9" size="1" layer="26" rot="MR90"/>
+</element>
+<element name="GND" library="OMAT_IC" package="SMD_ROUND_1.5MM" value="SMD_1.5MM" x="2.06" y="6.5" smashed="yes" rot="MR0">
+<attribute name="NAME" x="1.5" y="7.94" size="1" layer="26" rot="MR90"/>
+</element>
 </elements>
 <signals>
+<signal name="INT">
+<contactref element="INT" pad="1"/>
+</signal>
+<signal name="I2C_SDA">
+<contactref element="SDA" pad="1"/>
+</signal>
+<signal name="I2C_SCL">
+<contactref element="SCL" pad="1"/>
+</signal>
+<signal name="V33">
+<contactref element="V33" pad="1"/>
+</signal>
+<signal name="VCC">
+<contactref element="VCC" pad="1"/>
+</signal>
+<signal name="GND">
+<contactref element="GND" pad="1"/>
+<polygon width="0" layer="1">
+<vertex x="0" y="48"/>
+<vertex x="48" y="48"/>
+<vertex x="48" y="0"/>
+<vertex x="0" y="0"/>
+</polygon>
+<polygon width="0" layer="16">
+<vertex x="0" y="48"/>
+<vertex x="48" y="48"/>
+<vertex x="48" y="0"/>
+<vertex x="0" y="0"/>
+</polygon>
+<polygon width="0" layer="1">
+<vertex x="0" y="48"/>
+<vertex x="48" y="48"/>
+<vertex x="48" y="0"/>
+<vertex x="0" y="0"/>
+</polygon>
+</signal>
+<signal name="N$1">
+<polygon width="0" layer="16" pour="cutout" rank="2">
+<vertex x="43" y="13"/>
+<vertex x="43" y="30"/>
+<vertex x="12" y="30"/>
+<vertex x="12" y="13"/>
+</polygon>
+</signal>
 </signals>
 </board>

Commit message: some more work progress...
Parts:
- added C1, C2: (no value), rcl:C0603
- added D1: PCA9517-MSOP8, OMAT_IC:SOP65P490X110-8N
- added D2: AT24C02C-SOT23-5, Microchip_By_element14_Batch_1:SOT95P280X145-5N
- added N1: MCP1700T-1802E/TT, Microchip_By_element14_Batch_1:SOT95P237X112-3N
- added R1, R2: (no value), rcl:R0603
Connections:
- removed net I2C_SCL: SCL.1
- removed net I2C_SDA: SDA.1
- removed net V33: V33.1
- new net +1V8: C2.1, D1.1, D2.4, N1.2
- new net +3V3: C1.1, D1.8, N1.3, R1.2, R2.2, V33.1
- new net SCL_1V8: D1.2, D2.1, SCL.1
- new net SCL_3V3: D1.7, R1.1
- new net SDA_1V8: D1.3, D2.3, SDA.1
- new net SDA_3V3: D1.6, R2.1
- net GND: now also C1.2, C2.2, D1.4, D2.2, D2.5, N1.1
Routing:
- net +3V3: track 0.00 -> 37.8 mm, vias 0 -> 1
- net +1V8: track 0.00 -> 18.5 mm
- net SDA_1V8: track 0.00 -> 13.9 mm, vias 0 -> 1
- net GND: track 0.00 -> 10.7 mm, vias 0 -> 4
- net SCL_1V8: track 0.00 -> 10.3 mm, vias 0 -> 1
- net SDA_3V3: track 0.00 -> 5.33 mm
- net SCL_3V3: track 0.00 -> 3.41 mm
Other:
- outline, holes or cut-outs redrawn

Commit message: good night
Parts:
- added SCL_3V3, SDA_3V3, V18, _GND, _INT, _V33: SMD_1.5MM, OMAT_IC:SMD_ROUND_1.5MM
- added U$1: DAFUG, dafug:DAFUG
Connections:
- net +1V8: now also V18.1
- net +3V3: now also _V33.1
- net GND: now also _GND.1
- net INT: now also _INT.1
- net SCL_3V3: now also SCL_3V3.1
- net SDA_3V3: now also SDA_3V3.1
Routing:
- net INT: track 0.00 -> 41.8 mm, vias 0 -> 1
- net +1V8: track 18.5 -> 45.0 mm
- net SDA_3V3: track 5.33 -> 31.3 mm
- net SCL_3V3: track 3.41 -> 26.3 mm
- net +3V3: track 37.8 -> 48.5 mm
- net SDA_1V8: track 13.9 -> 14.6 mm
- net GND: vias 4 -> 13
Other:
- board text added: "(C) KIMMOLI 2013"
- board text added: "MY OTHER HALF"
- board text added: "V1.00"

Commit message: V1.00
Parts:
- added U$2: (no value), jollalogo:JOLLALOGO
Changed lines of the file:
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@@
 <setting verticaltext="up"/>
 </settings>
-<grid distance="0.2" unitdist="mm" unit="mm" style="lines" multiple="1" display="no" altdistance="0.025" altunitdist="inch" altunit="inch"/>
+<grid distance="2" unitdist="mil" unit="mil" style="lines" multiple="1" display="yes" altdistance="0.025" altunitdist="inch" altunit="inch"/>
 <layers>
 <layer number="1" name="Top" color="4" fill="1" visible="yes" active="yes"/>
@@
 <layer number="27" name="tValues" color="7" fill="1" visible="yes" active="yes"/>
 <layer number="28" name="bValues" color="7" fill="1" visible="yes" active="yes"/>
-<layer number="29" name="tStop" color="7" fill="3" visible="no" active="yes"/>
-<layer number="30" name="bStop" color="7" fill="6" visible="no" active="yes"/>
-<layer number="31" name="tCream" color="7" fill="4" visible="no" active="yes"/>
-<layer number="32" name="bCream" color="7" fill="5" visible="no" active="yes"/>
-<layer number="33" name="tFinish" color="6" fill="3" visible="no" active="yes"/>
-<layer number="34" name="bFinish" color="6" fill="6" visible="no" active="yes"/>
-<layer number="35" name="tGlue" color="7" fill="4" visible="no" active="yes"/>
-<layer number="36" name="bGlue" color="7" fill="5" visible="no" active="yes"/>
-<layer number="37" name="tTest" color="7" fill="1" visible="no" active="yes"/>
-<layer number="38" name="bTest" color="7" fill="1" visible="no" active="yes"/>
+<layer number="29" name="tStop" color="7" fill="3" visible="yes" active="yes"/>
+<layer number="30" name="bStop" color="7" fill="6" visible="yes" active="yes"/>
+<layer number="31" name="tCream" color="7" fill="4" visible="yes" active="yes"/>
+<layer number="32" name="bCream" color="7" fill="5" visible="yes" active="yes"/>
+<layer number="33" name="tFinish" color="6" fill="3" visible="yes" active="yes"/>
+<layer number="34" name="bFinish" color="6" fill="6" visible="yes" active="yes"/>
+<layer number="35" name="tGlue" color="7" fill="4" visible="yes" active="yes"/>
+<layer number="36" name="bGlue" color="7" fill="5" visible="yes" active="yes"/>
+<layer number="37" name="tTest" color="7" fill="1" visible="yes" active="yes"/>
+<layer number="38" name="bTest" color="7" fill="1" visible="yes" active="yes"/>
 <layer number="39" name="tKeepout" color="4" fill="11" visible="yes" active="yes"/>
 <layer number="40" name="bKeepout" color="1" fill="11" visible="yes" active="yes"/>
@@
 <layer number="42" name="bRestrict" color="1" fill="10" visible="yes" active="yes"/>
 <layer number="43" name="vRestrict" color="2" fill="10" visible="yes" active="yes"/>
-<layer number="44" name="Drills" color="7" fill="1" visible="no" active="yes"/>
+<layer number="44" name="Drills" color="7" fill="1" visible="yes" active="yes"/>
 <layer number="45" name="Holes" color="7" fill="1" visible="yes" active="yes"/>
-<layer number="46" name="Milling" color="3" fill="1" visible="no" active="yes"/>
-<layer number="47" name="Measures" color="7" fill="1" visible="no" active="yes"/>
+<layer number="46" name="Milling" color="3" fill="1" visible="yes" active="yes"/>
+<layer number="47" name="Measures" color="7" fill="1" visible="yes" active="yes"/>
 <layer number="48" name="Document" color="7" fill="1" visible="yes" active="yes"/>
 <layer number="49" name="Reference" color="7" fill="1" visible="yes" active="yes"/>
@@
 <attribute name="NAME" x="1.5" y="7.94" size="1" layer="26" rot="MR90"/>
 </element>
-<element name="D2" library="Microchip_By_element14_Batch_1" package="SOT95P280X145-5N" value="AT24C02C-SOT23-5" x="39.5" y="14.5" rot="R180">
+<element name="D2" library="Microchip_By_element14_Batch_1" package="SOT95P280X145-5N" value="AT24C02C-SOT23-5" x="39.5" y="14.5" smashed="yes" rot="R180">
 <attribute name="PACKAGE" value="SOT23-5" x="39.5" y="14.5" size="1.778" layer="27" rot="R180" display="off"/>
 <attribute name="OC_NEWARK" value="12C1993" x="39.5" y="14.5" size="1.778" layer="27" rot="R180" display="off"/>
@@
 <attribute name="SUPPLIER" value="MICROCHIP" x="39.5" y="14.5" size="1.778" layer="27" rot="R180" display="off"/>
 <attribute name="OC_FARNELL" value="9757880" x="39.5" y="14.5" size="1.778" layer="27" rot="R180" display="off"/>
-</element>
-<element name="D1" library="OMAT_IC" package="SOP65P490X110-8N" value="PCA9517-MSOP8" x="38.5" y="10" rot="R180"/>
-<element name="N1" library="Microchip_By_element14_Batch_1" package="SOT95P237X112-3N" value="MCP1700T-1802E/TT" x="43.3" y="21">
+<attribute name="NAME" x="41.7502" y="13.9796" size="1" layer="25" ratio="10" rot="SR0"/>
+<attribute name="VALUE" x="45.2658" y="18.4116" size="2.0828" layer="27" ratio="10" rot="SR180"/>
+</element>
+<element name="D1" library="OMAT_IC" package="SOP65P490X110-8N" value="PCA9517-MSOP8" x="38.5" y="10" smashed="yes" rot="R180">
+<attribute name="NAME" x="41.6456" y="8.94" size="1" layer="25" ratio="10" rot="SR0"/>
+<attribute name="VALUE" x="41.9544" y="14.445" size="2.0828" layer="27" ratio="10" rot="SR180"/>
+</element>
+<element name="N1" library="Microchip_By_element14_Batch_1" package="SOT95P237X112-3N" value="MCP1700T-1802E/TT" x="43.3" y="21" smashed="yes">
 <attribute name="PACKAGE" value="SOT23-3" x="43.3" y="21" size="1.778" layer="27" display="off"/>
 <attribute name="OC_NEWARK" value="84R5175" x="43.3" y="21" size="1.778" layer="27" display="off"/>
@@
 <attribute name="SUPPLIER" value="Microchip" x="43.3" y="21" size="1.778" layer="27" display="off"/>
 <attribute name="OC_FARNELL" value="1296591" x="43.3" y="21" size="1.778" layer="27" display="off"/>
-</element>
-<element name="C1" library="rcl" package="C0603" value="" x="40.8" y="21" rot="R270"/>
-<element name="C2" library="rcl" package="C0603" value="" x="45.8" y="21" rot="R90"/>
-<element name="R1" library="rcl" package="R0603" value="" x="37.7" y="6.7" rot="R270"/>
-<element name="R2" library="rcl" package="R0603" value="" x="39.7" y="6.7" rot="R270"/>
+<attribute name="NAME" x="42.3788" y="17.559" size="1" layer="25" ratio="10" rot="SR0"/>
+<attribute name="VALUE" x="37.839" y="16.7582" size="2.0828" layer="27" ratio="10" rot="SR0"/>
+</element>
+<element name="C1" library="rcl" package="C0603" value="" x="40.8" y="21" smashed="yes" rot="R270">
+<attribute name="NAME" x="39.765" y="18.235" size="1" layer="25"/>
+<attribute name="VALUE" x="38.895" y="21.635" size="0.8128" layer="27" rot="R270"/>
+</element>
+<element name="C2" library="rcl" package="C0603" value="" x="45.8" y="21" smashed="yes" rot="R90">
+<attribute name="NAME" x="46.635" y="19.365" size="1" layer="25" rot="R180"/>
+<attribute name="VALUE" x="47.705" y="20.365" size="0.8128" layer="27" rot="R90"/>
+</element>
+<element name="R1" library="rcl" package="R0603" value="" x="37.7" y="6.7" smashed="yes" rot="R270">
+<attribute name="NAME" x="35.065" y="6.335" size="1" layer="25"/>
+<attribute name="VALUE" x="35.795" y="7.335" size="0.8128" layer="27" rot="R270"/>
+</element>
+<element name="R2" library="rcl" package="R0603" value="" x="39.7" y="6.7" smashed="yes" rot="R270">
+<attribute name="NAME" x="40.665" y="6.335" size="1" layer="25"/>
+<attribute name="VALUE" x="37.795" y="7.335" size="0.8128" layer="27" rot="R270"/>
+</element>
 <element name="SCL_3V3" library="OMAT_IC" package="SMD_ROUND_1.5MM" value="SMD_1.5MM" x="17.54" y="3" smashed="yes">
 <attribute name="NAME" x="18" y="4.34" size="1" layer="25" rot="R90"/>
@@
 </element>
 <element name="U$1" library="dafug" package="DAFUG" value="DAFUG" x="5.8" y="42.2"/>
+<element name="U$2" library="jollalogo" package="JOLLALOGO" value="" x="15.0876" y="15.3924"/>
 </elements>
 <signals>
