File: myhalf.brd (EAGLE design)
At the start: 48 x 48 mm, 20 parts

Commit message: v1.10
Parts:
- removed SCL_3V3, SDA_3V3, V18, _GND, _INT, _V33: SMD_1.5MM, OMAT_IC:SMD_ROUND_1.5MM
- added H1: (no value), OMAT_IC:CHIP-LED0603
- added R3: 330, rcl:R0603
- added U$2: (no value), dafug:JOLLALOGO
- added X1: PIIKKIRIMA-10, OMAT_IC:PIIKKIRIMA-10
- R1, R2: value (none) -> 2K15
- moved D2 24.3 mm to (15.3, 12.0), turned to 0 degrees
- moved D1 16.5 mm to (22.1, 11.9), turned to 0 degrees
- moved C2 14.2 mm to (38.0, 9.10), turned to 180 degrees
- moved R2 12.5 mm to (28.4, 12.1), turned to 90 degrees
- moved N1 10.8 mm to (38.0, 11.7)
- moved C1 9.22 mm to (40.6, 11.8)
- moved R1 8.67 mm to (30.9, 12.1), turned to 90 degrees
- moved U$1 6.96 mm to (7.58, 35.5)
Connections:
- new net N$2: H1.A, R3.1
- net +1V8: now also X1.5; no longer V18.1
- net +3V3: now also R3.2, X1.2; no longer _V33.1
- net GND: now also H1.C, X1.1, X1.10; no longer _GND.1
- net INT: now also X1.6; no longer _INT.1
- net SCL_1V8: now also X1.7
- net SCL_3V3: now also X1.3; no longer SCL_3V3.1
- net SDA_1V8: now also X1.8
- net SDA_3V3: now also X1.4; no longer SDA_3V3.1
- net VCC: now also X1.9
Routing:
- net SDA_1V8: track 14.6 -> 57.9 mm, vias 1 -> 0
- net SCL_1V8: track 10.3 -> 49.3 mm, vias 1 -> 0
- net SDA_3V3: track 31.3 -> 8.84 mm
- net VCC: track 0.00 -> 15.3 mm
- net +3V3: track 48.5 -> 63.8 mm
- net GND: track 10.7 -> 0.00 mm, vias 13 -> 15
- net INT: track 41.8 -> 51.5 mm
- net SCL_3V3: track 26.3 -> 17.5 mm
- net N$2: track 0.00 -> 2.33 mm
Other:
- outline, holes or cut-outs redrawn
- board text added: "(C) KIMMOLI 2014"
- board text added: "+1V8"
- board text added: "+3V3"
- board text added: "GND"
- board text added: "INT~"
- board text added: "SCL1V8"
- board text added: "SCL3V3"
- board text added: "SDA1V8"
- board text added: "SDA3V3"
- board text added: "V1.10"
- board text added: "VCHG"
- board text removed: "(C) KIMMOLI 2013"
- board text removed: "V1.00"
